File: acoms_bec.brd (EAGLE design)
At the start: 50 x 40 mm, 9 parts, among them IC1 NJU7201L35, Q1 2SC2458, Q2 MJB45H11

Commit message: Transistor name update to the original
Parts:
- Q2: value MJB45H11 -> 2SB1318
Changed lines of the file:
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@@
 <attribute name="VALUE" x="12.7" y="14.732" size="1.27" layer="27" font="vector" ratio="10" rot="R180"/>
 </element>
-<element name="Q2" library="dp_devices" package="TO-92" value="MJB45H11" x="6.858" y="17.272" smashed="yes">
+<element name="Q2" library="dp_devices" package="TO-92" value="2SB1318" x="6.858" y="17.272" smashed="yes">
 <attribute name="NAME" x="4.318" y="20.32" size="1.27" layer="25" font="vector" ratio="10"/>
 <attribute name="VALUE" x="4.318" y="13.97" size="1.27" layer="27" font="vector" ratio="10"/>
